Commit message: feat: 区分竖装和平装livox 3d雷达

File: urdf/mid360_vertical.xacro (robot description, xacro)
@@ -6,10 +6,10 @@
   <xacro:property name="laser_max_range" value="80.0"/>
   <!-- 提高采样点数以获得更密集的点云 -->
-  <xacro:property name="samples" value="240000"/>
+  <xacro:property name="samples" value="20000"/>
   <!-- 提高分辨率以获得更好的点云质量 -->
-  <xacro:property name="resolution" value="0.001"/>
+  <xacro:property name="resolution" value="0.003"/>
   <xacro:property name="noise_mean" value="0.0"/>
   <!-- 适度降低噪声模拟以提高性能 -->
-  <xacro:property name="noise_stddev" value="0.01"/>
+  <xacro:property name="noise_stddev" value="0.005"/>
   <xacro:property name="mass" value="0.4" />
   <xacro:property name="length" value="0.1" />
@@ -23,5 +23,5 @@
     </inertial>
   </xacro:macro>
-  <xacro:macro name="mid360" params="name:='' parent:= 'base_link' topic:='mid360' *origin ">
+  <xacro:macro name="mid360_vertical" params="name:='' parent:= 'base_link' topic:='mid360_vertical' *origin ">
     <link name="${name}">
       <xacro:box_inertia m="${mass}" w="${width}" d="${length}" h="${height}"/>
@@ -58,5 +58,5 @@
 				<horizontal>
 				<!-- 提高水平采样点以获得更密集的水平扫描 -->
-				<samples>240</samples>
+				<samples>80</samples>
 				<resolution>1</resolution>
 				<min_angle>${0}</min_angle>
@@ -65,7 +65,7 @@
 				<vertical>
 				<!-- 提高垂直采样点以获得更密集的垂直扫描 -->
-				<samples>16</samples>
+				<samples>15</samples>
 				<resolution>1</resolution>
-				<min_angle>${-7/180*M_PI}</min_angle>
+				<min_angle>${0/180*M_PI}</min_angle>
 				<max_angle>${55.22/180*M_PI}</max_angle>
 				</vertical>
@@ -84,6 +84,6 @@
           <visualize>true</visualize>  <!-- 启用可视化以确保数据正常发布 -->
 		  <samples>${samples}</samples>
-		  <downsample>1</downsample>  <!-- 适度下采样以平衡性能和质量 -->
-		  <csv_file_name>$(find ros2_livox_simulation)/scan_mode/mid360.csv</csv_file_name>
+		  <downsample>10</downsample>  <!-- 适度下采样以平衡性能和质量 -->
+		  <csv_file_name>$(find ros2_livox_simulation)/scan_mode/mid360_vertical.csv</csv_file_name>
 		  <topic>${topic}</topic>
         </plugin>

Commit message: refactor: update logging configuration to use environment variables for log directory and filename; adjust noise standard deviation in URDF for performance improvement

File: urdf/mid360_vertical.xacro (robot description, xacro)
@@ -11,5 +11,5 @@
   <xacro:property name="noise_mean" value="0.0"/>
   <!-- 适度降低噪声模拟以提高性能 -->
-  <xacro:property name="noise_stddev" value="0.005"/>
+  <xacro:property name="noise_stddev" value="0.001"/>
   <xacro:property name="mass" value="0.4" />
   <xacro:property name="length" value="0.1" />
