Commit message: feat:使用mid360stl文件替代简单的盒子

File: urdf/mid360.xacro (robot description, xacro)
@@ -24,12 +24,20 @@
   </xacro:macro>
   <xacro:macro name="mid360" params="name:='' parent:= 'base_link' topic:='mid360' *origin ">
-<link name="${name}">
-<xacro:box_inertia m="${length}" w="${width}" d="${length}" h="${height}"/>
-  <visual>
+    <link name="${name}">
+      <xacro:box_inertia m="${mass}" w="${width}" d="${length}" h="${height}"/>
+      <visual>
         <geometry>
-            <box size="${length} ${width} ${height}"/>
+          <mesh filename="package://venice_robot_description/meshes/mid-360-asm.stl" scale="0.001 0.001 0.001"/>
         </geometry>
-  </visual>
-</link>
+        <material name="blue">
+          <color rgba="0 0 1 1"/>
+        </material>
+      </visual>
+      <collision>
+        <geometry>
+          <box size="${length} ${width} ${height}"/>
+        </geometry>
+      </collision>
+    </link>
     <joint name="${name}_joint" type="fixed">
       <parent link="${parent}"/>

Commit message: perf:调整仿真参数；添加cmake json输出方便插件工作

File: urdf/mid360.xacro (robot description, xacro)
@@ -6,5 +6,5 @@
   <xacro:property name="laser_max_range" value="80.0"/>
   <!-- 提高采样点数以获得更密集的点云 -->
-  <xacro:property name="samples" value="25000"/>
+  <xacro:property name="samples" value="20000"/>
   <!-- 提高分辨率以获得更好的点云质量 -->
   <xacro:property name="resolution" value="0.003"/>
@@ -50,5 +50,5 @@
         <visualize>true</visualize>
         <!-- 提高更新频率以获得更流畅的点云数据 -->
-        <update_rate>5</update_rate>
+        <update_rate>10</update_rate>
         <!-- This ray plgin is only for visualization. -->
         <plugin name="${name}_plugin" filename="libros2_livox.so">
@@ -83,5 +83,5 @@
           <visualize>true</visualize>  <!-- 启用可视化以确保数据正常发布 -->
 		  <samples>${samples}</samples>
-		  <downsample>2</downsample>  <!-- 适度下采样以平衡性能和质量 -->
+		  <downsample>10</downsample>  <!-- 适度下采样以平衡性能和质量 -->
 		  <csv_file_name>$(find ros2_livox_simulation)/scan_mode/mid360.csv</csv_file_name>
 		  <topic>${topic}</topic>

Commit message: feat: 增加竖装前置激光雷达/livox/lidar_vertical，之前雷达平装

File: urdf/mid360.xacro (robot description, xacro)
@@ -27,4 +27,5 @@
       <xacro:box_inertia m="${mass}" w="${width}" d="${length}" h="${height}"/>
       <visual>
+       <origin xyz="0 0 0" rpy="${M_PI/2} 0 ${M_PI}"/>
         <geometry>
           <mesh filename="package://venice_robot_description/meshes/mid-360-asm.stl" scale="0.001 0.001 0.001"/>

Commit message: feat: 每帧雷达等间隔覆盖CSV FOV

File: urdf/mid360.xacro (robot description, xacro)
@@ -6,5 +6,5 @@
   <xacro:property name="laser_max_range" value="80.0"/>
   <!-- 提高采样点数以获得更密集的点云 -->
-  <xacro:property name="samples" value="240000"/>
+  <xacro:property name="samples" value="24000"/>
   <!-- 提高分辨率以获得更好的点云质量 -->
   <xacro:property name="resolution" value="0.001"/>
@@ -84,5 +84,5 @@
           <visualize>true</visualize>  <!-- 启用可视化以确保数据正常发布 -->
 		  <samples>${samples}</samples>
-		  <downsample>1</downsample>  <!-- 适度下采样以平衡性能和质量 -->
+		  <downsample>2</downsample>  <!-- 适度下采样以平衡性能和质量 -->
 		  <csv_file_name>$(find ros2_livox_simulation)/scan_mode/mid360.csv</csv_file_name>
 		  <topic>${topic}</topic>

File: urdf/mid360_vertical.xacro (robot description, xacro)
@@ -6,5 +6,5 @@
   <xacro:property name="laser_max_range" value="80.0"/>
   <!-- 提高采样点数以获得更密集的点云 -->
-  <xacro:property name="samples" value="20000"/>
+  <xacro:property name="samples" value="10000"/>
   <!-- 提高分辨率以获得更好的点云质量 -->
   <xacro:property name="resolution" value="0.003"/>
@@ -58,5 +58,5 @@
 				<horizontal>
 				<!-- 提高水平采样点以获得更密集的水平扫描 -->
-				<samples>80</samples>
+				<samples>240</samples>
 				<resolution>1</resolution>
 				<min_angle>${0}</min_angle>
@@ -65,5 +65,5 @@
 				<vertical>
 				<!-- 提高垂直采样点以获得更密集的垂直扫描 -->
-				<samples>15</samples>
+				<samples>16</samples>
 				<resolution>1</resolution>
 				<min_angle>${0/180*M_PI}</min_angle>
@@ -84,5 +84,5 @@
           <visualize>true</visualize>  <!-- 启用可视化以确保数据正常发布 -->
 		  <samples>${samples}</samples>
-		  <downsample>10</downsample>  <!-- 适度下采样以平衡性能和质量 -->
+		  <downsample>1</downsample>  <!-- 适度下采样以平衡性能和质量 -->
 		  <csv_file_name>$(find ros2_livox_simulation)/scan_mode/mid360_vertical.csv</csv_file_name>
 		  <topic>${topic}</topic>

Commit message: feat: enhance livox point cloud message structure and update URDF parameters for improved lidar performance

File: urdf/mid360.xacro (robot description, xacro)
@@ -5,11 +5,10 @@
   <!-- 提高最大范围以获得更广的探测范围 -->
   <xacro:property name="laser_max_range" value="80.0"/>
-  <!-- 提高采样点数以获得更密集的点云 -->
-  <xacro:property name="samples" value="24000"/>
+  <!-- 每帧射线数 ≈ lidar_samples / lidar_downsample；过大则 CPU 跟不上，实际 Hz 会远低于 update_rate -->
   <!-- 提高分辨率以获得更好的点云质量 -->
-  <xacro:property name="resolution" value="0.001"/>
+  <!-- 与 mid360_vertical.xacro 分开命名，避免 venice 同时 include 时被覆盖 -->
+  <xacro:property name="mid360_range_resolution" value="0.001"/>
   <xacro:property name="noise_mean" value="0.0"/>
-  <!-- 适度降低噪声模拟以提高性能 -->
-  <xacro:property name="noise_stddev" value="0.01"/>
+  <xacro:property name="mid360_noise_stddev" value="0.01"/>
   <xacro:property name="mass" value="0.4" />
   <xacro:property name="length" value="0.1" />
@@ -23,5 +22,8 @@
     </inertial>
   </xacro:macro>
-  <xacro:macro name="mid360" params="name:='' parent:= 'base_link' topic:='mid360' *origin ">
+  <!-- publish_rate: 点云对外发布频率(Hz)，与 Gazebo update_rate 解耦；
+       lidar_samples/downsample 决定每帧射线数(越少→仿真越快→update_rate 越能跑满);
+       非重复扫描模式：每帧顺序推进 CSV 索引，经过足够帧后覆盖完整 FOV。 -->
+  <xacro:macro name="mid360" params="name:='' parent:= 'base_link' topic:='mid360' lidar_update_rate:=50 lidar_samples:=1500 lidar_downsample:=1 lidar_publish_rate:=15 *origin ">
     <link name="${name}">
       <xacro:box_inertia m="${mass}" w="${width}" d="${length}" h="${height}"/>
@@ -50,6 +52,6 @@
         <pose>0 0 0 0 0 0</pose>
         <visualize>true</visualize>
-        <!-- 提高更新频率以获得更流畅的点云数据 -->
-        <update_rate>10</update_rate>
+        <!-- Gazebo 传感器标称频率（Hz）；实际受物理步长与本帧射线计算耗时限制，改完需 colcon build ros2_livox_simulation -->
+        <update_rate>${lidar_update_rate}</update_rate>
         <!-- This ray plgin is only for visualization. -->
         <plugin name="${name}_plugin" filename="libros2_livox.so">
@@ -74,15 +76,17 @@
 				<min>${laser_min_range}</min>
 				<max>${laser_max_range}</max>
-				<resolution>${resolution}</resolution>
+				<resolution>${mid360_range_resolution}</resolution>
 			  </range>
 			  <noise>
 				<type>gaussian</type>
 				<mean>${noise_mean}</mean>
-				<stddev>${noise_stddev}</stddev>
+				<stddev>${mid360_noise_stddev}</stddev>
 			  </noise>
 			</ray>
           <visualize>true</visualize>  <!-- 启用可视化以确保数据正常发布 -->
-		  <samples>${samples}</samples>
-		  <downsample>2</downsample>  <!-- 适度下采样以平衡性能和质量 -->
+		  <samples>${lidar_samples}</samples>
+		  <downsample>${lidar_downsample}</downsample>
+		  <!-- 点云对外发布频率，与 Gazebo update_rate 解耦 -->
+		  <publish_rate>${lidar_publish_rate}</publish_rate>
 		  <csv_file_name>$(find ros2_livox_simulation)/scan_mode/mid360.csv</csv_file_name>
 		  <topic>${topic}</topic>

File: urdf/mid360_vertical.xacro (robot description, xacro)
@@ -5,11 +5,9 @@
   <!-- 提高最大范围以获得更广的探测范围 -->
   <xacro:property name="laser_max_range" value="80.0"/>
-  <!-- 提高采样点数以获得更密集的点云 -->
-  <xacro:property name="samples" value="10000"/>
+  <!-- 每帧射线数 ≈ lidar_samples / lidar_downsample；竖装雷达同样受 CPU 限制 -->
   <!-- 提高分辨率以获得更好的点云质量 -->
-  <xacro:property name="resolution" value="0.003"/>
+  <xacro:property name="mid360_vertical_range_resolution" value="0.003"/>
   <xacro:property name="noise_mean" value="0.0"/>
-  <!-- 适度降低噪声模拟以提高性能 -->
-  <xacro:property name="noise_stddev" value="0.001"/>
+  <xacro:property name="mid360_vertical_noise_stddev" value="0.001"/>
   <xacro:property name="mass" value="0.4" />
   <xacro:property name="length" value="0.1" />
@@ -23,5 +21,6 @@
     </inertial>
   </xacro:macro>
-  <xacro:macro name="mid360_vertical" params="name:='' parent:= 'base_link' topic:='mid360_vertical' *origin ">
+  <!-- publish_rate: 点云对外发布频率(Hz)，与 Gazebo update_rate 解耦 -->
+  <xacro:macro name="mid360_vertical" params="name:='' parent:= 'base_link' topic:='mid360_vertical' lidar_update_rate:=50 lidar_samples:=1500 lidar_downsample:=1 lidar_publish_rate:=15 *origin ">
     <link name="${name}">
       <xacro:box_inertia m="${mass}" w="${width}" d="${length}" h="${height}"/>
@@ -50,6 +49,5 @@
         <pose>0 0 0 0 0 0</pose>
         <visualize>true</visualize>
-        <!-- 提高更新频率以获得更流畅的点云数据 -->
-        <update_rate>10</update_rate>
+        <update_rate>${lidar_update_rate}</update_rate>
         <!-- This ray plgin is only for visualization. -->
         <plugin name="${name}_plugin" filename="libros2_livox.so">
@@ -74,15 +72,16 @@
 				<min>${laser_min_range}</min>
 				<max>${laser_max_range}</max>
-				<resolution>${resolution}</resolution>
+				<resolution>${mid360_vertical_range_resolution}</resolution>
 			  </range>
 			  <noise>
 				<type>gaussian</type>
 				<mean>${noise_mean}</mean>
-				<stddev>${noise_stddev}</stddev>
+				<stddev>${mid360_vertical_noise_stddev}</stddev>
 			  </noise>
 			</ray>
           <visualize>true</visualize>  <!-- 启用可视化以确保数据正常发布 -->
-		  <samples>${samples}</samples>
-		  <downsample>1</downsample>  <!-- 适度下采样以平衡性能和质量 -->
+		  <samples>${lidar_samples}</samples>
+		  <downsample>${lidar_downsample}</downsample>
+		  <publish_rate>${lidar_publish_rate}</publish_rate>
 		  <csv_file_name>$(find ros2_livox_simulation)/scan_mode/mid360_vertical.csv</csv_file_name>
 		  <topic>${topic}</topic>
