Commit message: feat: implement Gaussian noise configuration for range measurements in livox plugin and update URDF to support noise parameters

File: urdf/mid360.xacro (robot description, xacro)
@@ -10,5 +10,7 @@
   <xacro:property name="mid360_range_resolution" value="0.001"/>
   <xacro:property name="noise_mean" value="0.0"/>
-  <xacro:property name="mid360_noise_stddev" value="0.01"/>
+  <!-- 测距噪声：随 enable_sensor_noise 开关，默认 0（真值）；由 livox 插件读取 <noise> 并施加 -->
+  <xacro:arg name="enable_sensor_noise" default="false"/>
+  <xacro:property name="mid360_noise_stddev" value="${0.01 if '$(arg enable_sensor_noise)' == 'true' else 0.0}"/>
   <xacro:property name="mass" value="0.4" />
   <xacro:property name="length" value="0.1" />

File: urdf/mid360_vertical.xacro (robot description, xacro)
@@ -9,5 +9,7 @@
   <xacro:property name="mid360_vertical_range_resolution" value="0.003"/>
   <xacro:property name="noise_mean" value="0.0"/>
-  <xacro:property name="mid360_vertical_noise_stddev" value="0.001"/>
+  <!-- 测距噪声：随 enable_sensor_noise 开关，默认 0（真值）；由 livox 插件读取 <noise> 并施加 -->
+  <xacro:arg name="enable_sensor_noise" default="false"/>
+  <xacro:property name="mid360_vertical_noise_stddev" value="${0.001 if '$(arg enable_sensor_noise)' == 'true' else 0.0}"/>
   <xacro:property name="mass" value="0.4" />
   <xacro:property name="length" value="0.1" />
